Commit message: Removed gripper

File: urdf/ur_macro.xacro (robot description, xacro)
@@ -360,8 +360,4 @@
       <child link="${prefix}tool0"/>
     </joint>
-    <xacro:include filename="$(find soft_robotics_description)/urdf/soft_robotics_gripper.urdf.xacro" />
-    <xacro:soft_robotics_gripper prefix="${prefix}" parent="tool0" >
-    <origin xyz="0 0 0.004" rpy="0 ${-pi/2} ${pi}"/>
-  </xacro:soft_robotics_gripper>
   </xacro:macro>
 </robot>

Commit message: Fixed frames

File: urdf/ur_macro.xacro (robot description, xacro)
@@ -350,5 +350,5 @@
       <parent link="${prefix}wrist_3_link" />
       <child link="${prefix}flange" />
-      <origin xyz="0 0 0.16" rpy="0 ${-pi/2.0} ${-pi/2.0}" />
+      <origin xyz="0 0 0.1" rpy="0 ${-pi/2.0} ${-pi/2.0}" />
     </joint>
     <!-- ROS-Industrial 'tool0' frame - all-zeros tool frame -->
